File: christmas_bauble.kicad_pcb (KiCad board)
At the start: 2 copper layers, 110 x 110 mm, 50 parts, among them Q1 Q_NPN_EBC, Q2 Q_NPN_EBC, Q3 Q_NPN_EBC, Q4 Q_NPN_EBC, Q5 Q_NPN_EBC, SW1 SW_PUSH, SW2 SW_PUSH, SW3 SWITCH_INV, U1 595_SHIFT, U2 555

Commit message: Updating  stuff
Other:
- board text added: "Kookies Christmas Bauble Revision 2 Sep 2015"
- board text removed: "Kookies Christmas Bauble Revision 1.1 Sep 2015"
Changed lines of the file:
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@@
     (title "LED Christmas Bauble")
     (date 2015-09-12)
-    (rev 1.1)
+    (rev 2)
     (comment 1 "Adding coin battery and switching to SMD components")
   )
@@
     (visible_elements FFFEFFFF)
     (pcbplotparams
-      (layerselection 0x00030_80000001)
-      (usegerberextensions false)
+      (layerselection 0x01030_80000001)
+      (usegerberextensions true)
       (excludeedgelayer true)
       (linewidth 0.100000)
@@
     (fp_line (start -1.99898 23.50008) (end -1.09982 21.20138) (layer F.SilkS) (width 0.15))
   )
-  (gr_text "Kookies Christmas Bauble\nRevision 1.1\nSep 2015" (at 59.75 92) (layer F.SilkS)
+  (gr_text "Kookies Christmas Bauble\nRevision 2\nSep 2015" (at 59.75 92) (layer F.SilkS)
     (effects (font (size 1.5 1.5) (thickness 0.3)))
   )
