File: christmas_bauble_rev3.sch (KiCad schematic (older format))
At the start: 31 parts, among them SW1 SWITCH_INV, SW2 SW_PUSH, SW3 SW_PUSH, U1 LOGIC_SMD_XOR, U2 595_SHIFT, U3 555

Commit message: Changing batteries on the board to 2 20mm coin cell batteries in paralell for longer lifetime. Routing batteries on the back via SMD holders.
Parts:
- added BT2: Battery, kookie_utilities:20mm_coin_bat_smd, symbol Battery
- BT1: footprint kookie_utilities:COIN_BAT_HOLDER -> kookie_utilities:20mm_coin_bat_smd
- C1: footprint Capacitors_SMD:C_2225_HandSoldering -> SMD_Packages:SMD-1206_Pol
Connections:
- wire segments 96 -> 98
Changed lines of the file:
@@
 LIBS:contrib
 LIBS:valves
-LIBS:kookie_logic_symbols
-LIBS:christmas_bauble
 LIBS:christmas_bauble_rev3-cache
 EELAYER 25 0
@@
 F 0 "C1" H 8925 2200 50  0000 L CNN
 F 1 "22µF" H 8925 2000 50  0000 L CNN
-F 2 "Capacitors_SMD:C_2225_HandSoldering" H 8938 1950 30  0001 C CNN
+F 2 "SMD_Packages:SMD-1206_Pol" H 8938 1950 30  0001 C CNN
 F 3 "" H 8900 2100 60  0000 C CNN
 	1    8900 2100
@@
 F 0 "BT1" H 3350 3950 50  0000 L CNN
 F 1 "Battery" H 3350 3850 50  0000 L CNN
-F 2 "kookie_utilities:COIN_BAT_HOLDER" V 3250 3940 60  0001 C CNN
+F 2 "kookie_utilities:20mm_coin_bat_smd" V 3250 3940 60  0001 C CNN
 F 3 "" V 3250 3940 60  0000 C CNN
 	1    3250 3900
@@
 Wire Wire Line
 	2450 2700 2450 2850
+$Comp
+L Battery BT2
+U 1 1 564B077E
+P 2850 3900
+F 0 "BT2" H 2950 3950 50  0000 L CNN
+F 1 "Battery" H 2950 3850 50  0000 L CNN
+F 2 "kookie_utilities:20mm_coin_bat_smd" V 2850 3940 60  0001 C CNN
+F 3 "" V 2850 3940 60  0000 C CNN
+	1    2850 3900
+	1    0    0    -1
+$EndComp
+Wire Wire Line
+	2850 3750 2850 3700
+Connection ~ 2850 3700
+Wire Wire Line
+	2850 4050 2850 4150
+Connection ~ 2850 4150
 $EndSCHEMATC
